Commit message: updated urdf for real robot launch file

File: robotiq_description/urdf/robotiq_2f_85_gripper.urdf.xacro (robot description, xacro)
@@ -7,6 +7,6 @@
     <!-- Import macros -->
     <xacro:include filename="$(find robotiq_description)/urdf/robotiq_2f_85_macro.urdf.xacro" />
-    <link name="world" />
-    <xacro:robotiq_gripper name="RobotiqGripperHardwareInterface" prefix="$(arg prefix)" parent="world" use_fake_hardware="$(arg use_fake_hardware)" com_port="$(arg com_port)">
+    <link name="$(arg prefix)wrist_3_link" />
+    <xacro:robotiq_gripper name="RobotiqGripperHardwareInterface" prefix="$(arg prefix)" parent="$(arg prefix)wrist_3_link" use_fake_hardware="$(arg use_fake_hardware)" com_port="$(arg com_port)">
         <origin xyz="0 0 0" rpy="0 0 0" />
     </xacro:robotiq_gripper>
